Commit message: Figured out not to re-use key names for macro names, now have working robot_description

File: carbot_description/urdf/carbot.xacro (robot description, xacro)
@@ -1,11 +1,17 @@
 <?xml version="1.0"?>
 <robot name="carbot" xmlns:xacro="http://wiki.ros.org/xacro">
-<xacro:macro name="box" params="name length width height mass">
+<xacro:property name="car_length" value="1.4"/>
+<xacro:property name="car_width" value="1.0"/>
+<xacro:property name="car_height" value="0.3"/>
+<xacro:property name="wheel_width" value="0.2"/>
+<!-- don't use macro names that are the same as other key names
+  like 'box', 'cylinder', etc. otherwise get Invalid parameter "size"
+-->
+<xacro:macro name="block" params="name length width height mass">
   <link name="${name}">
-    <!--origin xyz="${length/2} ${width/2} ${height/2}" /-->
-    <visual>
-      <origin xyz="0 0 0" rpy="0 0 0" />
+     <visual>
+      <origin xyz="0 0 0" rpy="0 0 0"/>
       <geometry>
-        <box size="${length/2} ${width/2} ${height/2}"/>
+        <box size="${length} ${width} ${height}"/>
       </geometry>
       <material name="${name}_gray">
@@ -23,15 +29,15 @@
       <mass value="${mass}"/>
       <inertia
-          ixx="${mass / 12.0 * (width * width + height * height)" ixy="0.0" ixz="0.0"
-          iyy="${mass / 12.0 * (length * length + height * height)" iyz="0.0"
-          izz="${mass / 12.0 * (length * length + width * width)" />
+          ixx="${mass / 12.0 * (width * width + height * height)}" ixy="0.0" ixz="0.0"
+          iyy="${mass / 12.0 * (length * length + height * height)}" iyz="0.0"
+          izz="${mass / 12.0 * (length * length + width * width)}" />
     </inertial>
   </link>
 </xacro:macro>
 <!-- a wheel that rotates around the y axis, rolls forward toward the x axis -->
-<xacro:macro name="cylinder" params="name width height mass">
+<!--origin xyz="${length/2} ${width/2} ${height/2}" /-->
+<xacro:macro name="wheel" params="name width height mass">
   <link name="${name}">
     <visual>
-      <!--origin xyz="${length/2} ${width/2} ${height/2}" /-->
       <origin xyz="0 0 0" rpy="${pi/2} 0 0" />
       <geometry>
@@ -52,40 +58,41 @@
       <mass value="${mass}"/>
       <inertia
-          ixx="${mass / 12.0 * (3/4 * height * length + width * width)" ixy="0.0" ixz="0.0"
-          iyy="${mass / 12.0 * (3/4 * height * length + width * width)" iyz="0.0"
-          izz="${mass / 12.0 * (3/4 * height * length + width * width)"/>
+          ixx="${mass / 12.0 * (3/4 * height * height + width * width)}" ixy="0.0" ixz="0.0"
+          iyy="${mass / 12.0 * (3/4 * height * height + width * width)}" iyz="0.0"
+          izz="${mass / 12.0 * (3/4 * height * height + width * width)}"/>
     </inertial>
   </link>
 </xacro:macro>
-  <xacro:box name="base_link" length="1.0" width="0.6" height="0.2" mass="1.0"/>
-  <xacro:cylinder name="wheel_front_left" width="0.15" height="0.4" mass="0.2"/>
-  <joint name="wheel_front_left_axle">
+  <xacro:block name="base_link" length="${car_length}"
+      width="${car_width}" height="${car_height}" mass="1.0"/>
+  <xacro:wheel name="wheel_front_left" width="${wheel_width}" height="0.4" mass="0.2"/>
+  <joint name="wheel_front_left_axle" type="continuous">
     <parent link="base_link"/>
     <child link="wheel_front_left"/>
-    <origin xyz="0.3 0.32 0" rpy="0 0 "/>
+    <origin xyz="${car_length/2 - 0.05} ${car_width/2 + wheel_width/2 + 0.1} 0" rpy="0 0 0"/>
     <axis xyz="0 1 0"/>
     <limit effort="1000.0" velocity="0.5"/>
   </joint>
-  <xacro:cylinder name="wheel_front_right" width="0.15" height="0.4" mass="0.2"/>
-  <joint name="wheel_front_right">
+  <xacro:wheel name="wheel_front_right" width="${wheel_width}" height="0.4" mass="0.2"/>
+  <joint name="wheel_front_right" type="continuous">
     <parent link="base_link"/>
     <child link="wheel_front_right"/>
-    <origin xyz="0.3 -0.32 0" rpy="0 0 "/>
+    <origin xyz="${car_length/2 - 0.05} ${-1 * (car_width/2 + wheel_width/2 + 0.1)} 0" rpy="0 0 0"/>
     <axis xyz="0 -1 0"/>
     <limit effort="1000.0" velocity="0.5"/>
   </joint>
-  <xacro:cylinder name="wheel_back_left" width="0.15" height="0.4" mass="0.2"/>
-  <joint name="wheel_back_left_axle">
+  <xacro:wheel name="wheel_back_left" width="${wheel_width}" height="0.4" mass="0.2"/>
+  <joint name="wheel_back_left_axle" type="continuous">
     <parent link="base_link"/>
     <child link="wheel_back_left"/>
-    <origin xyz="-0.3 0.32 0" rpy="0 0 "/>
+    <origin xyz="${-car_length/2 + 0.05} ${car_width/2 + wheel_width/2 + 0.1} 0" rpy="0 0 0"/>
     <axis xyz="0 1 0"/>
     <limit effort="1000.0" velocity="0.5"/>
   </joint>
-  <xacro:cylinder name="wheel_back_right" width="0.15" height="0.4" mass="0.2"/>
-  <joint name="wheel_back_right_axle">
+  <xacro:wheel name="wheel_back_right" width="${wheel_width}" height="0.4" mass="0.2"/>
+  <joint name="wheel_back_right_axle" type="continuous">
     <parent link="base_link"/>
     <child link="wheel_back_right"/>
-    <origin xyz="-0.3 -0.32 0" rpy="0 0 "/>
+    <origin xyz="${-car_length/2 + 0.05} ${-1 * (car_width/2 + wheel_width/2 + 0.1)} 0" rpy="0 0 0"/>
     <axis xyz="0 -1 0"/>
     <limit effort="1000.0" velocity="0.5"/>

Commit message: The dependencies were causing problems when I had ros_comm in same directory, so commented them out

File: carbot_description/urdf/carbot.xacro (robot description, xacro)
@@ -66,9 +66,15 @@
   <xacro:block name="base_link" length="${car_length}"
       width="${car_width}" height="${car_height}" mass="1.0"/>
+  <link name="front_axle"/>
+  <joint name="front_axle_joint" type="fixed">
+    <parent link="base_link"/>
+    <child link="front_axle"/>
+    <origin xyz="${car_length/2 - 0.05} 0 0" rpy="0 0 0"/>
+  </joint>
   <xacro:wheel name="wheel_front_left" width="${wheel_width}" height="0.4" mass="0.2"/>
   <joint name="wheel_front_left_axle" type="continuous">
-    <parent link="base_link"/>
+    <parent link="front_axle"/>
     <child link="wheel_front_left"/>
-    <origin xyz="${car_length/2 - 0.05} ${car_width/2 + wheel_width/2 + 0.1} 0" rpy="0 0 0"/>
+    <origin xyz="0 ${car_width/2 + wheel_width/2 + 0.1} 0" rpy="0 0 0"/>
     <axis xyz="0 1 0"/>
     <limit effort="1000.0" velocity="0.5"/>
@@ -76,15 +82,21 @@
   <xacro:wheel name="wheel_front_right" width="${wheel_width}" height="0.4" mass="0.2"/>
   <joint name="wheel_front_right" type="continuous">
+    <parent link="front_axle"/>
+    <child link="wheel_front_right"/>
+    <origin xyz="0 ${-1 * (car_width/2 + wheel_width/2 + 0.1)} 0" rpy="0 0 0"/>
+    <axis xyz="0 1 0"/>
+    <limit effort="1000.0" velocity="0.5"/>
+  </joint>
+  <link name="back_axle"/>
+  <joint name="back_axle_joint" type="fixed">
     <parent link="base_link"/>
-    <child link="wheel_front_right"/>
-    <origin xyz="${car_length/2 - 0.05} ${-1 * (car_width/2 + wheel_width/2 + 0.1)} 0" rpy="0 0 0"/>
-    <axis xyz="0 -1 0"/>
-    <limit effort="1000.0" velocity="0.5"/>
+    <child link="back_axle"/>
+    <origin xyz="${-car_length/2 + 0.05} 0 0" rpy="0 0 0"/>
   </joint>
   <xacro:wheel name="wheel_back_left" width="${wheel_width}" height="0.4" mass="0.2"/>
   <joint name="wheel_back_left_axle" type="continuous">
-    <parent link="base_link"/>
+    <parent link="back_axle"/>
     <child link="wheel_back_left"/>
-    <origin xyz="${-car_length/2 + 0.05} ${car_width/2 + wheel_width/2 + 0.1} 0" rpy="0 0 0"/>
+    <origin xyz="0 ${car_width/2 + wheel_width/2 + 0.1} 0" rpy="0 0 0"/>
     <axis xyz="0 1 0"/>
     <limit effort="1000.0" velocity="0.5"/>
@@ -92,8 +104,8 @@
   <xacro:wheel name="wheel_back_right" width="${wheel_width}" height="0.4" mass="0.2"/>
   <joint name="wheel_back_right_axle" type="continuous">
-    <parent link="base_link"/>
+    <parent link="back_axle"/>
     <child link="wheel_back_right"/>
-    <origin xyz="${-car_length/2 + 0.05} ${-1 * (car_width/2 + wheel_width/2 + 0.1)} 0" rpy="0 0 0"/>
-    <axis xyz="0 -1 0"/>
+    <origin xyz="0 ${-1 * (car_width/2 + wheel_width/2 + 0.1)} 0" rpy="0 0 0"/>
+    <axis xyz="0 1 0"/>
     <limit effort="1000.0" velocity="0.5"/>
   </joint>

Commit message: Now the front wheels can steer

File: carbot_description/urdf/carbot.xacro (robot description, xacro)
@@ -72,17 +72,33 @@
     <origin xyz="${car_length/2 - 0.05} 0 0" rpy="0 0 0"/>
   </joint>
+  <link name="front_left_steer"/>
+  <joint name="front_left_steer_joint" type="revolute">
+    <parent link="front_axle"/>
+    <child link="front_left_steer"/>
+    <origin xyz="0 ${car_width/2 + wheel_width/2 + 0.1} 0" rpy="0 0 0"/>
+    <axis xyz="0 0 -1"/>
+    <limit effort="1000.0" upper="0.7" lower="-0.7" velocity="0.5"/>
+  </joint>
   <xacro:wheel name="wheel_front_left" width="${wheel_width}" height="0.4" mass="0.2"/>
   <joint name="wheel_front_left_axle" type="continuous">
-    <parent link="front_axle"/>
+    <parent link="front_left_steer"/>
     <child link="wheel_front_left"/>
-    <origin xyz="0 ${car_width/2 + wheel_width/2 + 0.1} 0" rpy="0 0 0"/>
+    <origin xyz="0 0 0" rpy="0 0 0"/>
     <axis xyz="0 1 0"/>
     <limit effort="1000.0" velocity="0.5"/>
   </joint>
+  <link name="front_right_steer"/>
+  <joint name="front_right_steer_joint" type="revolute">
+    <parent link="front_axle"/>
+    <child link="front_right_steer"/>
+    <origin xyz="0 ${-car_width/2 - wheel_width/2 - 0.1} 0" rpy="0 0 0"/>
+    <axis xyz="0 0 -1"/>
+    <limit effort="1000.0" upper="0.7" lower="-0.7" velocity="0.5"/>
+  </joint>
   <xacro:wheel name="wheel_front_right" width="${wheel_width}" height="0.4" mass="0.2"/>
   <joint name="wheel_front_right" type="continuous">
-    <parent link="front_axle"/>
+    <parent link="front_right_steer"/>
     <child link="wheel_front_right"/>
-    <origin xyz="0 ${-1 * (car_width/2 + wheel_width/2 + 0.1)} 0" rpy="0 0 0"/>
+    <origin xyz="0 0 0" rpy="0 0 0"/>
     <axis xyz="0 1 0"/>
     <limit effort="1000.0" velocity="0.5"/>

Commit message: Now am visualizing the spin center- later make this a marker that is a line from the steer link to the spin center.

File: carbot_description/urdf/carbot.xacro (robot description, xacro)
@@ -72,4 +72,16 @@
     <origin xyz="${car_length/2 - 0.05} 0 0" rpy="0 0 0"/>
   </joint>
+  <!-- this is the virtual joint that represents the front of the bicycle
+    in the bicycle model, it will be controlled and the left and right
+    actual joints will respond to it appropriately to maintain a steer center
+    -->
+  <link name="front_steer"/>
+  <joint name="front_steer_joint" type="revolute">
+    <parent link="front_axle"/>
+    <child link="front_steer"/>
+    <origin xyz="0 0.5 0" rpy="0 0 0"/>
+    <axis xyz="0 0 -1"/>
+    <limit effort="1000.0" upper="0.7" lower="-0.7" velocity="0.5"/>
+  </joint>
   <link name="front_left_steer"/>
   <joint name="front_left_steer_joint" type="revolute">

Commit message: This acker steering works for turning left, but the angle jumps all over when turning right

File: carbot_description/urdf/carbot.xacro (robot description, xacro)
@@ -80,5 +80,5 @@
     <parent link="front_axle"/>
     <child link="front_steer"/>
-    <origin xyz="0 0.5 0" rpy="0 0 0"/>
+    <origin xyz="0 0 0" rpy="0 0 0"/>
     <axis xyz="0 0 -1"/>
     <limit effort="1000.0" upper="0.7" lower="-0.7" velocity="0.5"/>

Commit message: Show the trajectory for all wheels, including the virtual one, and start incorporating velocity.  It isn't clear whether this node should be the odometry source but it is convenient for now to store all the acker calculations here.

File: carbot_description/urdf/carbot.xacro (robot description, xacro)
@@ -76,12 +76,28 @@
     actual joints will respond to it appropriately to maintain a steer center
     -->
-  <link name="front_steer"/>
-  <joint name="front_steer_joint" type="revolute">
+  <link name="lead_steer"/>
+  <joint name="lead_steer_joint" type="revolute">
+    <!-- TODO(lwalter) may want to put this at base_link instead- but
+      maybe thinking about moving in terms of where to put the front
+      bumper makes more sense than where to put the center of the vehicle?
+      -->
+    <!--parent link="base_link"/-->
     <parent link="front_axle"/>
-    <child link="front_steer"/>
+    <child link="lead_steer"/>
     <origin xyz="0 0 0" rpy="0 0 0"/>
     <axis xyz="0 0 -1"/>
     <limit effort="1000.0" upper="0.7" lower="-0.7" velocity="0.5"/>
   </joint>
+  <!-- virtual wheel that will represent the desired velocity
+    of the vehicle (so need radius encoded in it also) -->
+  <link name="wheel_lead"/>
+  <joint name="wheel_lead_axle" type="continuous">
+    <parent link="lead_steer"/>
+    <child link="wheel_lead"/>
+    <origin xyz="0 0 0" rpy="0 0 0"/>
+    <axis xyz="0 1 0"/>
+    <limit effort="1000.0" velocity="0.5"/>
+  </joint>
+  <!-- front left -->
   <link name="front_left_steer"/>
   <joint name="front_left_steer_joint" type="revolute">
@@ -100,4 +116,5 @@
     <limit effort="1000.0" velocity="0.5"/>
   </joint>
+  <!-- front right -->
   <link name="front_right_steer"/>
   <joint name="front_right_steer_joint" type="revolute">
@@ -109,5 +126,5 @@
   </joint>
   <xacro:wheel name="wheel_front_right" width="${wheel_width}" height="0.4" mass="0.2"/>
-  <joint name="wheel_front_right" type="continuous">
+  <joint name="wheel_front_right_axle" type="continuous">
     <parent link="front_right_steer"/>
     <child link="wheel_front_right"/>
@@ -122,17 +139,30 @@
     <origin xyz="${-car_length/2 + 0.05} 0 0" rpy="0 0 0"/>
   </joint>
+  <!-- back left -->
+  <link name="back_left"/>
+  <joint name="back_left_axle" type="fixed">
+    <parent link="back_axle"/>
+    <child link="back_left"/>
+    <origin xyz="0 ${car_width/2 + wheel_width/2 + 0.1} 0" rpy="0 0 0"/>
+  </joint>
   <xacro:wheel name="wheel_back_left" width="${wheel_width}" height="0.4" mass="0.2"/>
   <joint name="wheel_back_left_axle" type="continuous">
-    <parent link="back_axle"/>
+    <parent link="back_left"/>
     <child link="wheel_back_left"/>
-    <origin xyz="0 ${car_width/2 + wheel_width/2 + 0.1} 0" rpy="0 0 0"/>
+    <origin xyz="0 0 0" rpy="0 0 0"/>
     <axis xyz="0 1 0"/>
     <limit effort="1000.0" velocity="0.5"/>
   </joint>
+  <link name="back_right"/>
+  <joint name="back_right_axle" type="fixed">
+    <parent link="back_axle"/>
+    <child link="back_right"/>
+    <origin xyz="0 ${-1 * (car_width/2 + wheel_width/2 + 0.1)} 0" rpy="0 0 0"/>
+  </joint>
   <xacro:wheel name="wheel_back_right" width="${wheel_width}" height="0.4" mass="0.2"/>
   <joint name="wheel_back_right_axle" type="continuous">
-    <parent link="back_axle"/>
+    <parent link="back_right"/>
     <child link="wheel_back_right"/>
-    <origin xyz="0 ${-1 * (car_width/2 + wheel_width/2 + 0.1)} 0" rpy="0 0 0"/>
+    <origin xyz="0 0 0" rpy="0 0 0"/>
     <axis xyz="0 1 0"/>
     <limit effort="1000.0" velocity="0.5"/>

Commit message: Untested changes, still haven't calculated proper steer angle from linear x y

File: carbot_description/urdf/carbot.xacro (robot description, xacro)
@@ -5,4 +5,9 @@
 <xacro:property name="car_height" value="0.3"/>
 <xacro:property name="wheel_width" value="0.2"/>
+<!-- TODO(lwalter) pass these in as args -->
+<!-- turning to left -->
+<xacro:property name="min_steer" value="-0.7"/>
+<!-- turning to right -->
+<xacro:property name="max_steer" value="0.7"/>
 <!-- don't use macro names that are the same as other key names
   like 'box', 'cylinder', etc. otherwise get Invalid parameter "size"
@@ -87,5 +92,5 @@
     <origin xyz="0 0 0" rpy="0 0 0"/>
     <axis xyz="0 0 -1"/>
-    <limit effort="1000.0" upper="0.7" lower="-0.7" velocity="0.5"/>
+    <limit effort="1000.0" upper="${max_steer}" lower="${min_steer}" velocity="0.5"/>
   </joint>
   <!-- virtual wheel that will represent the desired velocity
@@ -106,5 +111,5 @@
     <origin xyz="0 ${car_width/2 + wheel_width/2 + 0.1} 0" rpy="0 0 0"/>
     <axis xyz="0 0 -1"/>
-    <limit effort="1000.0" upper="0.7" lower="-0.7" velocity="0.5"/>
+    <limit effort="1000.0" upper="${max_steer}" lower="${min_steer}" velocity="0.5"/>
   </joint>
   <xacro:wheel name="wheel_front_left" width="${wheel_width}" height="0.4" mass="0.2"/>
@@ -123,5 +128,5 @@
     <origin xyz="0 ${-car_width/2 - wheel_width/2 - 0.1} 0" rpy="0 0 0"/>
     <axis xyz="0 0 -1"/>
-    <limit effort="1000.0" upper="0.7" lower="-0.7" velocity="0.5"/>
+    <limit effort="1000.0" upper="${max_steer}" lower="${min_steer}" velocity="0.5"/>
   </joint>
   <xacro:wheel name="wheel_front_right" width="${wheel_width}" height="0.4" mass="0.2"/>

Commit message: Now that all intermediate links have inertia, the whole robot appears in gazebo

File: carbot_description/urdf/carbot.xacro (robot description, xacro)
@@ -10,4 +10,5 @@
 <!-- turning to right -->
 <xacro:property name="max_steer" value="0.7"/>
+<xacro:include filename="$(find carbot_description)/urdf/carbot.gazebo"/>
 <!-- don't use macro names that are the same as other key names
   like 'box', 'cylinder', etc. otherwise get Invalid parameter "size"
@@ -27,5 +28,5 @@
       <origin xyz="0 0 0" rpy="0 0 0" />
       <geometry>
-        <box size="${length/2} ${width/2} ${height/2}"/>
+        <box size="${length} ${width} ${height}"/>
       </geometry>
     </collision>
@@ -69,7 +70,21 @@
   </link>
 </xacro:macro>
-  <xacro:block name="base_link" length="${car_length}"
+  <link name="base_link"/>
+  <xacro:block name="chassis_link" length="${car_length}"
       width="${car_width}" height="${car_height}" mass="1.0"/>
-  <link name="front_axle"/>
+  <joint name="chassis_joint" type="fixed">
+    <parent link="base_link"/>
+    <child link="chassis_link"/>
+    <origin xyz="0 0 0" rpy="0 0 0"/>
+  </joint>
+  <xacro:block name="test_link" length="${car_length/2.0}"
+      width="${car_width}" height="${car_height}" mass="0.5"/>
+  <joint name="test_joint" type="fixed">
+    <parent link="base_link"/>
+    <child link="test_link"/>
+    <origin xyz="0 0 ${car_height}" rpy="0 0 0"/>
+  </joint>
+  <xacro:block name="front_axle" length="${car_width/8.0}"
+      width="${car_width}" height="${car_width/8.0}" mass="0.1"/>
   <joint name="front_axle_joint" type="fixed">
     <parent link="base_link"/>
@@ -105,5 +120,6 @@
   </joint>
   <!-- front left -->
-  <link name="front_left_steer"/>
+  <xacro:block name="front_left_steer" length="${car_width/8.0}"
+      width="${car_width/8.0}" height="${car_width/8.0}" mass="0.1"/>
   <joint name="front_left_steer_joint" type="revolute">
     <parent link="front_axle"/>
@@ -122,5 +138,6 @@
   </joint>
   <!-- front right -->
-  <link name="front_right_steer"/>
+  <xacro:block name="front_right_steer" length="${car_width/8.0}"
+      width="${car_width/8.0}" height="${car_width/8.0}" mass="0.1"/>
   <joint name="front_right_steer_joint" type="revolute">
     <parent link="front_axle"/>
@@ -138,5 +155,6 @@
     <limit effort="1000.0" velocity="0.5"/>
   </joint>
-  <link name="back_axle"/>
+  <xacro:block name="back_axle" length="${car_width/8.0}"
+      width="${car_width}" height="${car_width/8.0}" mass="0.1"/>
   <joint name="back_axle_joint" type="fixed">
     <parent link="base_link"/>
@@ -145,5 +163,6 @@
   </joint>
   <!-- back left -->
-  <link name="back_left"/>
+  <xacro:block name="back_left" length="${car_width/8.0}"
+      width="${car_width/8.0}" height="${car_width/8.0}" mass="0.1"/>
   <joint name="back_left_axle" type="fixed">
     <parent link="back_axle"/>
@@ -159,5 +178,6 @@
     <limit effort="1000.0" velocity="0.5"/>
   </joint>
-  <link name="back_right"/>
+  <xacro:block name="back_right" length="${car_width/8.0}"
+      width="${car_width/8.0}" height="${car_width/8.0}" mass="0.1"/>
   <joint name="back_right_axle" type="fixed">
     <parent link="back_axle"/>
