Commit message: macro-ized the steerable and fixed wheels, also creating a base_link steer joint that the cmd_vel or acker script needs to set.

File: carbot_description/urdf/carbot.xacro (robot description, xacro)
@@ -70,4 +70,40 @@
   </link>
 </xacro:macro>
+<xacro:macro name="fixed_wheel" params="name parent y">
+  <xacro:block name="${name}" length="${car_width/8.0}"
+      width="${car_width/8.0}" height="${car_width/8.0}" mass="0.1"/>
+  <joint name="${name}_axle" type="fixed">
+    <parent link="${parent}"/>
+    <child link="${name}"/>
+    <origin xyz="0 ${y} 0" rpy="0 0 0"/>
+  </joint>
+  <xacro:wheel name="wheel_${name}" width="${wheel_width}" height="0.4" mass="0.2"/>
+  <joint name="wheel_${name}_axle" type="continuous">
+    <parent link="${name}"/>
+    <child link="wheel_${name}"/>
+    <origin xyz="0 0 0" rpy="0 0 0"/>
+    <axis xyz="0 1 0"/>
+    <limit effort="1000.0" velocity="0.5"/>
+  </joint>
+</xacro:macro>
+<xacro:macro name="steered_wheel" params="name parent y">
+  <xacro:block name="${name}_steer" length="${car_width/8.0}"
+      width="${car_width/8.0}" height="${car_width/8.0}" mass="0.1"/>
+  <joint name="${name}_steer_joint" type="revolute">
+    <parent link="${parent}"/>
+    <child link="${name}_steer"/>
+    <origin xyz="0 ${y} 0" rpy="0 0 0"/>
+    <axis xyz="0 0 -1"/>
+    <limit effort="1000.0" upper="${max_steer}" lower="${min_steer}" velocity="0.5"/>
+  </joint>
+  <xacro:wheel name="wheel_${name}" width="${wheel_width}" height="0.4" mass="0.2"/>
+  <joint name="wheel_${name}_axle" type="continuous">
+    <parent link="${name}_steer"/>
+    <child link="wheel_${name}"/>
+    <origin xyz="0 0 0" rpy="0 0 0"/>
+    <axis xyz="0 1 0"/>
+    <limit effort="1000.0" velocity="0.5"/>
+  </joint>
+</xacro:macro>
   <link name="base_link"/>
   <xacro:block name="chassis_link" length="${car_length}"
@@ -78,4 +114,16 @@
     <origin xyz="0 0 0" rpy="0 0 0"/>
   </joint>
+  <!-- virtual joint that allows visualization of where the
+    base_link is steering (given the lead steer joint)
+    -->
+  <link name="base_steer"/>
+  <joint name="base_steer_joint" type="revolute">
+    <!--parent link="base_link"/-->
+    <parent link="base_link"/>
+    <child link="base_steer"/>
+    <origin xyz="0 0 0" rpy="0 0 0"/>
+    <axis xyz="0 0 -1"/>
+    <limit effort="1000.0" upper="${max_steer}" lower="${min_steer}" velocity="0.5"/>
+  </joint>
   <xacro:block name="test_link" length="${car_length/2.0}"
       width="${car_width}" height="${car_height}" mass="0.5"/>
@@ -85,4 +133,8 @@
     <origin xyz="0 0 ${car_height}" rpy="0 0 0"/>
   </joint>
+  <!-- every link has to have inertia in order for it to work in gazebo
+    even if it just connects two inertia links- without it the child link
+    that doesn't have inertia won't appear.
+    -->
   <xacro:block name="front_axle" length="${car_width/8.0}"
       width="${car_width}" height="${car_width/8.0}" mass="0.1"/>
@@ -119,40 +171,8 @@
     <limit effort="1000.0" velocity="0.5"/>
   </joint>
-  <!-- front left -->
-  <xacro:block name="front_left_steer" length="${car_width/8.0}"
-      width="${car_width/8.0}" height="${car_width/8.0}" mass="0.1"/>
-  <joint name="front_left_steer_joint" type="revolute">
-    <parent link="front_axle"/>
-    <child link="front_left_steer"/>
-    <origin xyz="0 ${car_width/2 + wheel_width/2 + 0.1} 0" rpy="0 0 0"/>
-    <axis xyz="0 0 -1"/>
-    <limit effort="1000.0" upper="${max_steer}" lower="${min_steer}" velocity="0.5"/>
-  </joint>
-  <xacro:wheel name="wheel_front_left" width="${wheel_width}" height="0.4" mass="0.2"/>
-  <joint name="wheel_front_left_axle" type="continuous">
-    <parent link="front_left_steer"/>
-    <child link="wheel_front_left"/>
-    <origin xyz="0 0 0" rpy="0 0 0"/>
-    <axis xyz="0 1 0"/>
-    <limit effort="1000.0" velocity="0.5"/>
-  </joint>
-  <!-- front right -->
-  <xacro:block name="front_right_steer" length="${car_width/8.0}"
-      width="${car_width/8.0}" height="${car_width/8.0}" mass="0.1"/>
-  <joint name="front_right_steer_joint" type="revolute">
-    <parent link="front_axle"/>
-    <child link="front_right_steer"/>
-    <origin xyz="0 ${-car_width/2 - wheel_width/2 - 0.1} 0" rpy="0 0 0"/>
-    <axis xyz="0 0 -1"/>
-    <limit effort="1000.0" upper="${max_steer}" lower="${min_steer}" velocity="0.5"/>
-  </joint>
-  <xacro:wheel name="wheel_front_right" width="${wheel_width}" height="0.4" mass="0.2"/>
-  <joint name="wheel_front_right_axle" type="continuous">
-    <parent link="front_right_steer"/>
-    <child link="wheel_front_right"/>
-    <origin xyz="0 0 0" rpy="0 0 0"/>
-    <axis xyz="0 1 0"/>
-    <limit effort="1000.0" velocity="0.5"/>
-  </joint>
+  <xacro:steered_wheel name="front_left" parent="front_axle"
+      y="${car_width/2 + wheel_width/2 + 0.1}"/>
+  <xacro:steered_wheel name="front_right" parent="front_axle"
+      y="${-car_width/2 - wheel_width/2 - 0.1}"/>
   <xacro:block name="back_axle" length="${car_width/8.0}"
       width="${car_width}" height="${car_width/8.0}" mass="0.1"/>
@@ -162,34 +182,7 @@
     <origin xyz="${-car_length/2 + 0.05} 0 0" rpy="0 0 0"/>
   </joint>
-  <!-- back left -->
-  <xacro:block name="back_left" length="${car_width/8.0}"
-      width="${car_width/8.0}" height="${car_width/8.0}" mass="0.1"/>
-  <joint name="back_left_axle" type="fixed">
-    <parent link="back_axle"/>
-    <child link="back_left"/>
-    <origin xyz="0 ${car_width/2 + wheel_width/2 + 0.1} 0" rpy="0 0 0"/>
-  </joint>
-  <xacro:wheel name="wheel_back_left" width="${wheel_width}" height="0.4" mass="0.2"/>
-  <joint name="wheel_back_left_axle" type="continuous">
-    <parent link="back_left"/>
-    <child link="wheel_back_left"/>
-    <origin xyz="0 0 0" rpy="0 0 0"/>
-    <axis xyz="0 1 0"/>
-    <limit effort="1000.0" velocity="0.5"/>
-  </joint>
-  <xacro:block name="back_right" length="${car_width/8.0}"
-      width="${car_width/8.0}" height="${car_width/8.0}" mass="0.1"/>
-  <joint name="back_right_axle" type="fixed">
-    <parent link="back_axle"/>
-    <child link="back_right"/>
-    <origin xyz="0 ${-1 * (car_width/2 + wheel_width/2 + 0.1)} 0" rpy="0 0 0"/>
-  </joint>
-  <xacro:wheel name="wheel_back_right" width="${wheel_width}" height="0.4" mass="0.2"/>
-  <joint name="wheel_back_right_axle" type="continuous">
-    <parent link="back_right"/>
-    <child link="wheel_back_right"/>
-    <origin xyz="0 0 0" rpy="0 0 0"/>
-    <axis xyz="0 1 0"/>
-    <limit effort="1000.0" velocity="0.5"/>
-  </joint>
+  <xacro:fixed_wheel name="back_left" parent="back_axle"
+      y="${car_width/2 + wheel_width/2 + 0.1}"/>
+  <xacro:fixed_wheel name="back_right" parent="back_axle"
+      y="${-1 * (car_width/2 + wheel_width/2 + 0.1)}"/>
 </robot>

Commit message: Untested transmissions for every steerable joint and wheel, untested controllers for just steering so far

File: carbot_description/urdf/carbot.xacro (robot description, xacro)
@@ -70,4 +70,6 @@
   </link>
 </xacro:macro>
+<!-- TODO(lucasw) make a wheel xacro to get common code out of
+    fixed_wheel and steered_wheel -->
 <xacro:macro name="fixed_wheel" params="name parent y">
   <xacro:block name="${name}" length="${car_width/8.0}"
@@ -86,4 +88,14 @@
     <limit effort="1000.0" velocity="0.5"/>
   </joint>
+  <transmission name="${name}_tran">
+    <type>transmission_interface/SimpleTransmission</type>
+    <joint name="${name}_joint">
+      <hardwareInterface>VelocityJointInterface</hardwareInterface>
+    </joint>
+    <actuator name="${name}_motor">
+      <hardwareInterface>VelocityJointInterface</hardwareInterface>
+      <mechanicalReduction>1</mechanicalReduction>
+    </actuator>
+  </transmission>
 </xacro:macro>
 <xacro:macro name="steered_wheel" params="name parent y">
@@ -97,4 +109,14 @@
     <limit effort="1000.0" upper="${max_steer}" lower="${min_steer}" velocity="0.5"/>
   </joint>
+  <transmission name="${name}_steer_tran">
+    <type>transmission_interface/SimpleTransmission</type>
+    <joint name="${name}_steer_joint">
+      <hardwareInterface>PositionJointInterface</hardwareInterface>
+    </joint>
+    <actuator name="${name}_steer_motor">
+      <hardwareInterface>PositionJointInterface</hardwareInterface>
+      <mechanicalReduction>1</mechanicalReduction>
+    </actuator>
+  </transmission>
   <xacro:wheel name="wheel_${name}" width="${wheel_width}" height="0.4" mass="0.2"/>
   <joint name="wheel_${name}_axle" type="continuous">
@@ -105,4 +127,15 @@
     <limit effort="1000.0" velocity="0.5"/>
   </joint>
+  <!-- TODO(lucasw) make front wheel drive optional -->
+  <transmission name="${name}_tran">
+    <type>transmission_interface/SimpleTransmission</type>
+    <joint name="${name}_joint">
+      <hardwareInterface>VelocityJointInterface</hardwareInterface>
+    </joint>
+    <actuator name="${name}_motor">
+      <hardwareInterface>VelocityJointInterface</hardwareInterface>
+      <mechanicalReduction>1</mechanicalReduction>
+    </actuator>
+  </transmission>
 </xacro:macro>
   <link name="base_link"/>

Commit message: Now have gazebo controller controlling the steer joints, but have disabled the acker script control- that needs to publish to the command topic rather than setting the joint state directly, optionally.  If the gazebo controller doesn't support desired position and velocity then it will probably be inadequate in the future, a custom gazebo plugin would be required?

File: carbot_description/urdf/carbot.xacro (robot description, xacro)
@@ -90,9 +90,9 @@
   <transmission name="${name}_tran">
     <type>transmission_interface/SimpleTransmission</type>
-    <joint name="${name}_joint">
-      <hardwareInterface>VelocityJointInterface</hardwareInterface>
+    <joint name="wheel_${name}_axle">
+      <hardwareInterface>EffortJointInterface</hardwareInterface>
     </joint>
     <actuator name="${name}_motor">
-      <hardwareInterface>VelocityJointInterface</hardwareInterface>
+      <hardwareInterface>EffortJointInterface</hardwareInterface>
       <mechanicalReduction>1</mechanicalReduction>
     </actuator>
@@ -112,8 +112,8 @@
     <type>transmission_interface/SimpleTransmission</type>
     <joint name="${name}_steer_joint">
-      <hardwareInterface>PositionJointInterface</hardwareInterface>
+      <hardwareInterface>EffortJointInterface</hardwareInterface>
     </joint>
     <actuator name="${name}_steer_motor">
-      <hardwareInterface>PositionJointInterface</hardwareInterface>
+      <hardwareInterface>EffortJointInterface</hardwareInterface>
       <mechanicalReduction>1</mechanicalReduction>
     </actuator>
@@ -130,9 +130,9 @@
   <transmission name="${name}_tran">
     <type>transmission_interface/SimpleTransmission</type>
-    <joint name="${name}_joint">
-      <hardwareInterface>VelocityJointInterface</hardwareInterface>
+    <joint name="wheel_${name}_axle">
+      <hardwareInterface>EffortJointInterface</hardwareInterface>
     </joint>
-    <actuator name="${name}_motor">
-      <hardwareInterface>VelocityJointInterface</hardwareInterface>
+    <actuator name="wheel_${name}_motor">
+      <hardwareInterface>EffortJointInterface</hardwareInterface>
       <mechanicalReduction>1</mechanicalReduction>
     </actuator>

Commit message: Trying out joystick with carbot, realize now that cmd vel interpretation is wrong- need to use only linear x and angular z, can't do any linear y.

File: carbot_description/urdf/carbot.xacro (robot description, xacro)
@@ -100,5 +100,7 @@
   <gazebo reference="wheel_${name}">
     <mu1>800</mu1>
-    <mu2>800</mu2>
+    <mu2>100</mu2>
+    <kp value="10000000.0"/>
+    <kd value="1.0"/>
   </gazebo>
 </xacro:macro>
@@ -145,5 +147,5 @@
   <link name="base_link"/>
   <xacro:block name="chassis_link" length="${car_length}"
-      width="${car_width}" height="${car_height}" mass="1.0"/>
+      width="${car_width}" height="${car_height}" mass="10.0"/>
   <joint name="chassis_joint" type="fixed">
     <parent link="base_link"/>
@@ -168,5 +170,5 @@
     <parent link="base_link"/>
     <child link="test_link"/>
-    <origin xyz="0 0 ${car_height}" rpy="0 0 0"/>
+    <origin xyz="0.1 0 ${car_height}" rpy="0 0 0"/>
   </joint>
   <!-- every link has to have inertia in order for it to work in gazebo

Commit message: More instructions, also trying to tune wheels and steering pid

File: carbot_description/urdf/carbot.xacro (robot description, xacro)
@@ -86,5 +86,5 @@
     <origin xyz="0 0 0" rpy="0 0 0"/>
     <axis xyz="0 1 0"/>
-    <limit effort="1000.0" velocity="0.5"/>
+    <limit effort="100.0" velocity="0.5"/>
   </joint>
   <transmission name="${name}_tran">
@@ -113,5 +113,5 @@
     <origin xyz="0 ${y} 0" rpy="0 0 0"/>
     <axis xyz="0 0 -1"/>
-    <limit effort="1000.0" upper="${max_steer}" lower="${min_steer}" velocity="0.5"/>
+    <limit effort="10.0" upper="${max_steer}" lower="${min_steer}" velocity="0.5"/>
   </joint>
   <transmission name="${name}_steer_tran">

Commit message: Now have onboard camera, and wheel spinning indicators.

File: carbot_description/urdf/carbot.xacro (robot description, xacro)
@@ -4,5 +4,6 @@
 <xacro:property name="car_width" value="1.0"/>
 <xacro:property name="car_height" value="0.3"/>
-<xacro:property name="wheel_width" value="0.2"/>
+<xacro:property name="wheel_width" value="0.15"/>
+<xacro:property name="wheel_radius" value="0.2"/>
 <!-- TODO(lwalter) pass these in as args -->
 <!-- turning to left -->
@@ -14,5 +15,5 @@
   like 'box', 'cylinder', etc. otherwise get Invalid parameter "size"
 -->
-<xacro:macro name="block" params="name length width height mass">
+<xacro:macro name="block" params="name length width height mass r:=0.5 b:=0.5 g:=0.5">
   <link name="${name}">
      <visual>
@@ -22,5 +23,5 @@
       </geometry>
       <material name="${name}_gray">
-        <color rgba="0.5 0.5 0.5 1"/>
+        <color rgba="${r} ${g} ${b} 1"/>
       </material>
     </visual>
@@ -43,10 +44,10 @@
 <!-- a wheel that rotates around the y axis, rolls forward toward the x axis -->
 <!--origin xyz="${length/2} ${width/2} ${height/2}" /-->
-<xacro:macro name="wheel" params="name width height mass">
+<xacro:macro name="wheel" params="name width radius mass">
   <link name="${name}">
     <visual>
       <origin xyz="0 0 0" rpy="${pi/2} 0 0" />
       <geometry>
-        <cylinder length="${width}" radius="${height/2}"/>
+        <cylinder length="${width}" radius="${radius}"/>
       </geometry>
       <material name="${name}_black">
@@ -57,5 +58,5 @@
       <origin xyz="0 0 0" rpy="${pi/2} 0 0" />
       <geometry>
-        <cylinder length="${width}" radius="${height/2}"/>
+        <cylinder length="${width}" radius="${radius}"/>
       </geometry>
     </collision>
@@ -64,7 +65,7 @@
       <mass value="${mass}"/>
       <inertia
-          ixx="${mass / 12.0 * (3/4 * height * height + width * width)}" ixy="0.0" ixz="0.0"
-          iyy="${mass / 12.0 * (3/4 * height * height + width * width)}" iyz="0.0"
-          izz="${mass / 12.0 * (3/4 * height * height + width * width)}"/>
+          ixx="${mass / 12.0 * (3 * radius * radius + width * width)}" ixy="0.0" ixz="0.0"
+          iyy="${mass / 12.0 * (3 * radius * radius + width * width)}" iyz="0.0"
+          izz="${mass / 2.0 * (radius * radius)}"/>
     </inertial>
   </link>
@@ -80,11 +81,20 @@
     <origin xyz="0 ${y} 0" rpy="0 0 0"/>
   </joint>
-  <xacro:wheel name="wheel_${name}" width="${wheel_width}" height="0.4" mass="0.2"/>
+  <xacro:wheel name="wheel_${name}" width="${wheel_width}" radius="${wheel_radius}" mass="0.2"/>
   <joint name="wheel_${name}_axle" type="continuous">
     <parent link="${name}"/>
     <child link="wheel_${name}"/>
-    <origin xyz="0 0 0" rpy="0 0 0"/>
+    <origin xyz="0 0 ${-car_height/4}" rpy="0 0 0"/>
     <axis xyz="0 1 0"/>
     <limit effort="100.0" velocity="0.5"/>
+  </joint>
+  <!-- indicate whether the wheel is spinning -->
+  <xacro:block name="wheel_${name}_hubcap" length="${1.6 * wheel_radius}"
+      width="${1.1 * wheel_width}" height="${0.2 * wheel_width}" mass="0.1"
+      r="0.95" g="0.95" b="0.95"/>
+  <joint name="wheel_${name}_hubcap_joint" type="fixed">
+    <parent link="wheel_${name}"/>
+    <child link="wheel_${name}_hubcap"/>
+    <origin xyz="0 0 0" rpy="0 0 0"/>
   </joint>
   <transmission name="${name}_tran">
@@ -125,9 +135,9 @@
     </actuator>
   </transmission>
-  <xacro:wheel name="wheel_${name}" width="${wheel_width}" height="0.4" mass="0.2"/>
+  <xacro:wheel name="wheel_${name}" width="${wheel_width}" radius="0.2" mass="1.0"/>
   <joint name="wheel_${name}_axle" type="continuous">
     <parent link="${name}_steer"/>
     <child link="wheel_${name}"/>
-    <origin xyz="0 0 0" rpy="0 0 0"/>
+    <origin xyz="0 0 ${-car_height/4}" rpy="0 0 0"/>
     <axis xyz="0 1 0"/>
     <limit effort="1000.0" velocity="0.5"/>
@@ -165,10 +175,10 @@
     <limit effort="1000.0" upper="${max_steer}" lower="${min_steer}" velocity="0.5"/>
   </joint>
-  <xacro:block name="test_link" length="${car_length/2.0}"
-      width="${car_width}" height="${car_height}" mass="0.5"/>
+  <xacro:block name="top_link" length="${car_length/2.0}"
+      width="${0.8 * car_width}" height="${0.9 * car_height}" mass="0.5"/>
   <joint name="test_joint" type="fixed">
     <parent link="base_link"/>
-    <child link="test_link"/>
-    <origin xyz="0.1 0 ${car_height}" rpy="0 0 0"/>
+    <child link="top_link"/>
+    <origin xyz="-0.1 0 ${car_height * 0.7}" rpy="0 0 0"/>
   </joint>
   <!-- every link has to have inertia in order for it to work in gazebo
@@ -181,5 +191,5 @@
     <parent link="base_link"/>
     <child link="front_axle"/>
-    <origin xyz="${car_length/2 - 0.05} 0 0" rpy="0 0 0"/>
+    <origin xyz="${car_length/2 - 0.1} 0 0" rpy="0 0 0"/>
   </joint>
   <!-- this is the virtual joint that represents the front of the bicycle
@@ -219,5 +229,5 @@
     <parent link="base_link"/>
     <child link="back_axle"/>
-    <origin xyz="${-car_length/2 + 0.05} 0 0" rpy="0 0 0"/>
+    <origin xyz="${-car_length/2 + 0.1} 0 0" rpy="0 0 0"/>
   </joint>
   <xacro:fixed_wheel name="back_left" parent="back_axle"
@@ -225,3 +235,21 @@
   <xacro:fixed_wheel name="back_right" parent="back_axle"
       y="${-1 * (car_width/2 + wheel_width/2 + 0.1)}"/>
+  <!-- sensors -->
+  <xacro:block name="camera_link" length="0.05"
+      width="0.04" height="0.03" mass="0.1"/>
+  <joint name="camera_joint" type="fixed">
+    <parent link="base_link"/>
+    <child link="camera_link"/>
+    <origin xyz="0.1 0 0.5" rpy="0 0.15 0"/>
+  </joint>
+  <link name="camera_link_optical"/>
+  <!-- generate an optical frame http://www.ros.org/reps/rep-0103.html#suffix-frames
+      so that ros and opencv can operate on the camera frame correctly -->
+  <joint name="camera_optical_joint" type="fixed">
+    <!-- these values have to be these values otherwise the gazebo camera image
+        won't be aligned properly with the frame it is supposedly originating from -->
+    <origin xyz="0 0 0" rpy="${-pi/2} 0 ${-pi/2}"/>
+    <parent link="camera_link"/>
+    <child link="camera_link_optical"/>
+  </joint>
 </robot>
