Commit message: Made common wheel code into xacro block

File: carbot_description/urdf/carbot.xacro (robot description, xacro)
@@ -71,4 +71,39 @@
   </link>
 </xacro:macro>
+<xacro:macro name="generic_wheel" params="name parent radius width">
+  <xacro:wheel name="wheel_${name}" width="${wheel_width}" radius="${wheel_radius}" mass="0.2"/>
+  <joint name="wheel_${name}_axle" type="continuous">
+    <parent link="${parent}"/>
+    <child link="wheel_${name}"/>
+    <origin xyz="0 0 ${-car_height/4}" rpy="0 0 0"/>
+    <axis xyz="0 1 0"/>
+    <limit effort="100.0" velocity="0.5"/>
+  </joint>
+  <!-- indicate whether the wheel is spinning -->
+  <xacro:block name="wheel_${name}_hubcap" length="${1.6 * wheel_radius}"
+      width="${1.1 * wheel_width}" height="${0.2 * wheel_width}" mass="0.1"
+      r="0.95" g="0.95" b="0.95"/>
+  <joint name="wheel_${name}_hubcap_joint" type="fixed">
+    <parent link="wheel_${name}"/>
+    <child link="wheel_${name}_hubcap"/>
+    <origin xyz="0 0 0" rpy="0 0 0"/>
+  </joint>
+  <transmission name="${name}_tran">
+    <type>transmission_interface/SimpleTransmission</type>
+    <joint name="wheel_${name}_axle">
+      <hardwareInterface>EffortJointInterface</hardwareInterface>
+    </joint>
+    <actuator name="${name}_motor">
+      <hardwareInterface>EffortJointInterface</hardwareInterface>
+      <mechanicalReduction>1</mechanicalReduction>
+    </actuator>
+  </transmission>
+  <gazebo reference="wheel_${name}">
+    <mu1>800</mu1>
+    <mu2>100</mu2>
+    <kp value="10000000.0"/>
+    <kd value="1.0"/>
+  </gazebo>
+</xacro:macro>  <!-- generic wheel -->
 <!-- TODO(lucasw) make a wheel xacro to get common code out of
     fixed_wheel and steered_wheel -->
@@ -81,37 +116,6 @@
     <origin xyz="0 ${y} 0" rpy="0 0 0"/>
   </joint>
-  <xacro:wheel name="wheel_${name}" width="${wheel_width}" radius="${wheel_radius}" mass="0.2"/>
-  <joint name="wheel_${name}_axle" type="continuous">
-    <parent link="${name}"/>
-    <child link="wheel_${name}"/>
-    <origin xyz="0 0 ${-car_height/4}" rpy="0 0 0"/>
-    <axis xyz="0 1 0"/>
-    <limit effort="100.0" velocity="0.5"/>
-  </joint>
-  <!-- indicate whether the wheel is spinning -->
-  <xacro:block name="wheel_${name}_hubcap" length="${1.6 * wheel_radius}"
-      width="${1.1 * wheel_width}" height="${0.2 * wheel_width}" mass="0.1"
-      r="0.95" g="0.95" b="0.95"/>
-  <joint name="wheel_${name}_hubcap_joint" type="fixed">
-    <parent link="wheel_${name}"/>
-    <child link="wheel_${name}_hubcap"/>
-    <origin xyz="0 0 0" rpy="0 0 0"/>
-  </joint>
-  <transmission name="${name}_tran">
-    <type>transmission_interface/SimpleTransmission</type>
-    <joint name="wheel_${name}_axle">
-      <hardwareInterface>EffortJointInterface</hardwareInterface>
-    </joint>
-    <actuator name="${name}_motor">
-      <hardwareInterface>EffortJointInterface</hardwareInterface>
-      <mechanicalReduction>1</mechanicalReduction>
-    </actuator>
-  </transmission>
-  <gazebo reference="wheel_${name}">
-    <mu1>800</mu1>
-    <mu2>100</mu2>
-    <kp value="10000000.0"/>
-    <kd value="1.0"/>
-  </gazebo>
+  <xacro:generic_wheel name="${name}" parent="${name}"
+      radius="${wheel_radius}" width="${wheel_width}"/>
 </xacro:macro>
 <xacro:macro name="steered_wheel" params="name parent y">
@@ -135,23 +139,6 @@
     </actuator>
   </transmission>
-  <xacro:wheel name="wheel_${name}" width="${wheel_width}" radius="0.2" mass="1.0"/>
-  <joint name="wheel_${name}_axle" type="continuous">
-    <parent link="${name}_steer"/>
-    <child link="wheel_${name}"/>
-    <origin xyz="0 0 ${-car_height/4}" rpy="0 0 0"/>
-    <axis xyz="0 1 0"/>
-    <limit effort="1000.0" velocity="0.5"/>
-  </joint>
-  <!-- TODO(lucasw) make front wheel drive optional -->
-  <transmission name="${name}_tran">
-    <type>transmission_interface/SimpleTransmission</type>
-    <joint name="wheel_${name}_axle">
-      <hardwareInterface>EffortJointInterface</hardwareInterface>
-    </joint>
-    <actuator name="wheel_${name}_motor">
-      <hardwareInterface>EffortJointInterface</hardwareInterface>
-      <mechanicalReduction>1</mechanicalReduction>
-    </actuator>
-  </transmission>
+  <xacro:generic_wheel name="${name}" parent="${name}_steer"
+      radius="${wheel_radius}" width="${wheel_width}"/>
 </xacro:macro>
   <link name="base_link"/>

Commit message: Making camera higher up and more pointed down so it can see the wheels steer

File: carbot_description/urdf/carbot.xacro (robot description, xacro)
@@ -228,5 +228,5 @@
     <parent link="base_link"/>
     <child link="camera_link"/>
-    <origin xyz="0.1 0 0.5" rpy="0 0.15 0"/>
+    <origin xyz="0.1 0 0.8" rpy="0 0.4 0"/>
   </joint>
   <link name="camera_link_optical"/>

Commit message: Have a prismatic joint to raise and lower camera, mostly to have an example prismatic joint

File: carbot_description/urdf/carbot.xacro (robot description, xacro)
@@ -223,10 +223,19 @@
       y="${-1 * (car_width/2 + wheel_width/2 + 0.1)}"/>
   <!-- sensors -->
+  <xacro:block name="camera_mast" length="0.04"
+      width="0.02" height="0.03" mass="0.1"/>
+  <joint name="camera_mast_joint" type="prismatic">
+    <parent link="base_link"/>
+    <child link="camera_mast"/>
+    <origin xyz="0.1 0 0.4" rpy="0 0 0"/>
+    <axis xyz="0 0 1"/>
+    <limit effort="20.0" velocity="0.25" lower="0.0" upper="0.5"/>
+  </joint>
   <xacro:block name="camera_link" length="0.05"
       width="0.04" height="0.03" mass="0.1"/>
   <joint name="camera_joint" type="fixed">
-    <parent link="base_link"/>
+    <parent link="camera_mast"/>
     <child link="camera_link"/>
-    <origin xyz="0.1 0 0.8" rpy="0 0.4 0"/>
+    <origin xyz="0.0 0 0.0" rpy="0 0.4 0"/>
   </joint>
   <link name="camera_link_optical"/>
